File: hardware/BREAD_Slice.kicad_pcb (KiCad board)
At the start: 2 copper layers, 70 x 100 mm, 16 parts, among them J1 I2C_01x04, J2 Conn_01x10_Female

Commit message: added opamps
Parts:
- removed the J1 at (150.2, 136.4)
- added NT1: NetTie_2, NetTie:NetTie-2_SMD_Pad2.0mm, B.Cu at (128.7, 115.2)
- HS1: footprint KML-Custom:Thermal Pad -> kml-custom:Thermal Pad
- U1: value ~ -> AP63205
- moved A1 2.56 mm to (142.6, 97.4)
- moved Logo1 1.57 mm to (128.2, 71.9)
- moved HS1 0.46 mm to (131.8, 121.5)
- moved D1 0.45 mm to (173.1, 135.7)
- moved C1 0.25 mm to (128.8, 119.5)
- moved C4 0.05 mm to (133.8, 116.4)
- renumbered J2 to J1
Connections:
- net /E_STOP renamed /ESTOP
- J1 pad 1: GND -> GNDPWR
- J1 pad 10: GND -> GNDPWR
- J1 pad 5: GND -> GNDPWR
Routing:
- net GNDPWR: track 0.00 -> 43.7 mm
- net /LED: track 51.5 -> 92.9 mm
- net /I2C_CLK: track 72.3 -> 46.3 mm, vias 2 -> 0
- net /I2C_DAT: track 70.5 -> 46.0 mm, vias 2 -> 0
- net /ESTOP: track 30.1 -> 23.6 mm
- net /INT: track 28.8 -> 23.3 mm
- net +5V: track 108.9 -> 104.2 mm
- net /SYNC: track 27.9 -> 23.7 mm
- net GND: track 19.6 -> 16.8 mm, vias 14 -> 20
- net +12V: track 46.8 -> 48.2 mm
- added copper zone on B.Cu, net GNDPWR
Other:
- outline, holes or cut-outs redrawn
- board text added: "BREAD Slice Template SLC_TEMP R3 04-2025"
- board text removed: "5V I2C Connector"
- board text removed: "BREAD Slice Template SLC_TEMP <version> <year>"

Commit message: finalized initial schematic and board
Parts:
- added C10: 10n, Capacitor_SMD:C_0603_1608Metric_Pad1.08x0.95mm_HandSolder, F.Cu at (156.8, 68.5)
- added C11: 1u, Capacitor_SMD:C_0603_1608Metric_Pad1.08x0.95mm_HandSolder, F.Cu at (155.8, 82.9)
- added C12: 1u, Capacitor_SMD:C_0603_1608Metric_Pad1.08x0.95mm_HandSolder, F.Cu at (158.1, 87.8)
- added C13: 0.22u, Capacitor_SMD:C_0603_1608Metric_Pad1.08x0.95mm_HandSolder, F.Cu at (155.8, 84.5)
- added C14: 0.22u, Capacitor_SMD:C_0603_1608Metric_Pad1.08x0.95mm_HandSolder, F.Cu at (158.1, 89.5)
- added C15: 10n, Capacitor_SMD:C_0603_1608Metric_Pad1.08x0.95mm_HandSolder, F.Cu at (156.8, 75.3)
- added C16: 10n, Capacitor_SMD:C_0603_1608Metric_Pad1.08x0.95mm_HandSolder, F.Cu at (156.8, 78.7)
- added C17: 10n, Capacitor_SMD:C_0603_1608Metric_Pad1.08x0.95mm_HandSolder, F.Cu at (177.4, 109.2)
- added C18: 10u, Capacitor_SMD:C_0805_2012Metric_Pad1.18x1.45mm_HandSolder, F.Cu at (173.7, 110.2)
- added C19: 10n, Capacitor_SMD:C_0603_1608Metric_Pad1.08x0.95mm_HandSolder, F.Cu at (177.5, 99.5)
- added C20: 10u, Capacitor_SMD:C_0805_2012Metric_Pad1.18x1.45mm_HandSolder, F.Cu at (173.7, 98.5)
- added C21: 0.1u, Capacitor_SMD:C_0603_1608Metric_Pad1.08x0.95mm_HandSolder, F.Cu at (171.8, 110.1)
- added C22: 0.1u, Capacitor_SMD:C_0603_1608Metric_Pad1.08x0.95mm_HandSolder, F.Cu at (171.8, 98.7)
- added C23: 0.1u, Capacitor_SMD:C_0603_1608Metric_Pad1.08x0.95mm_HandSolder, F.Cu at (178.2, 113.5)
- added C24: 0.1u, Capacitor_SMD:C_0603_1608Metric_Pad1.08x0.95mm_HandSolder, F.Cu at (178.3, 95.3)
- added C25: 10u X7R, Capacitor_SMD:C_1206_3216Metric_Pad1.33x1.80mm_HandSolder, F.Cu at (136.0, 80.8)
- added C26: 10n X7R, Capacitor_SMD:C_0603_1608Metric_Pad1.08x0.95mm_HandSolder, F.Cu at (134.0, 85.7)
- added C27: 10n X7R, Capacitor_SMD:C_0603_1608Metric_Pad1.08x0.95mm_HandSolder, F.Cu at (145.4, 84.7)
- added C28: 10u X7R, Capacitor_SMD:C_1206_3216Metric_Pad1.33x1.80mm_HandSolder, F.Cu at (147.1, 89.5)
- added C5: 1u, Capacitor_SMD:C_0603_1608Metric_Pad1.08x0.95mm_HandSolder, F.Cu at (155.2, 61.4)
- added C6: 1u, Capacitor_SMD:C_0603_1608Metric_Pad1.08x0.95mm_HandSolder, F.Cu at (155.2, 64.9)
- added C7: 0.22u, Capacitor_SMD:C_0603_1608Metric_Pad1.08x0.95mm_HandSolder, F.Cu at (153.6, 61.4)
- added C8: 0.22u, Capacitor_SMD:C_0603_1608Metric_Pad1.08x0.95mm_HandSolder, F.Cu at (153.6, 64.9)
- added C9: 10n, Capacitor_SMD:C_0603_1608Metric_Pad1.08x0.95mm_HandSolder, F.Cu at (156.8, 71.9)
- added D10: DF2S6.8MFS_L3M, Diode_SMD:D_SOD-923, F.Cu at (182.6, 79.2)
- added D11: DF2S6.8MFS_L3M, Diode_SMD:D_SOD-923, F.Cu at (182.7, 85.0)
- added D12: DF2S6.8MFS_L3M, Diode_SMD:D_SOD-923, F.Cu at (183.0, 105.0)
- added D13: DF2S6.8MFS_L3M, Diode_SMD:D_SOD-923, F.Cu at (183.0, 109.3)
- added D14: DF2S6.8MFS_L3M, Diode_SMD:D_SOD-923, F.Cu at (183.0, 99.7)
- added D15: DF2S6.8MFS_L3M, Diode_SMD:D_SOD-923, F.Cu at (183.0, 103.8)
- added D8: DF2S6.8MFS_L3M, Diode_SMD:D_SOD-923, F.Cu at (182.6, 67.7)
- added D9: DF2S6.8MFS_L3M, Diode_SMD:D_SOD-923, F.Cu at (182.6, 73.5)
- added J2: Conn_01x02, Connector_Molex:Molex_PicoBlade_53048-0210_1x02_P1.25mm_Horizontal, F.Cu at (186.0, 66.1)
- added J3: Conn_01x02, Connector_Molex:Molex_PicoBlade_53048-0210_1x02_P1.25mm_Horizontal, F.Cu at (186.0, 71.9)
- added J4: Conn_01x02, Connector_Molex:Molex_PicoBlade_53048-0210_1x02_P1.25mm_Horizontal, F.Cu at (186.0, 77.7)
- added J5: Conn_01x02, Connector_Molex:Molex_PicoBlade_53048-0210_1x02_P1.25mm_Horizontal, F.Cu at (186.0, 83.5)
- added J6: Conn_01x02, Connector_Molex:Molex_PicoBlade_53048-0210_1x02_P1.25mm_Horizontal, F.Cu at (186.0, 107.8)
- added J7: Conn_01x02, Connector_Molex:Molex_PicoBlade_53048-0210_1x02_P1.25mm_Horizontal, F.Cu at (186.0, 102.1)
- added NT2: NetTie_2, NetTie:NetTie-2_SMD_Pad2.0mm, F.Cu at (139.9, 90.1)
- added Q1: BC858BWT1G, Package_TO_SOT_SMD:SOT-323_SC-70, F.Cu at (182.4, 65.3)
- added Q2: BSS806NH6327XTSA1, Package_TO_SOT_SMD:SOT-23, F.Cu at (179.0, 65.3)
- added Q3: BC858BWT1G, Package_TO_SOT_SMD:SOT-323_SC-70, F.Cu at (182.4, 71.1)
- added Q4: BSS806NH6327XTSA1, Package_TO_SOT_SMD:SOT-23, F.Cu at (179.0, 71.1)
- added Q5: BC858BWT1G, Package_TO_SOT_SMD:SOT-323_SC-70, F.Cu at (182.4, 76.9)
- added Q6: BSS806NH6327XTSA1, Package_TO_SOT_SMD:SOT-23, F.Cu at (179.0, 76.9)
- added Q7: BC858BWT1G, Package_TO_SOT_SMD:SOT-323_SC-70, F.Cu at (182.4, 82.8)
- added Q8: BSS806NH6327XTSA1, Package_TO_SOT_SMD:SOT-23, F.Cu at (179.1, 82.8)
- added R1: 3.3k 1%, Resistor_SMD:R_0603_1608Metric_Pad0.98x0.95mm_HandSolder, F.Cu at (150.9, 62.4)
- added R10: 200k 1%, Resistor_SMD:R_0603_1608Metric_Pad0.98x0.95mm_HandSolder, F.Cu at (168.2, 71.2)
- added R11: 1k 1%, Resistor_SMD:R_0603_1608Metric_Pad0.98x0.95mm_HandSolder, F.Cu at (166.6, 67.7)
- added R12: 1k 1%, Resistor_SMD:R_0603_1608Metric_Pad0.98x0.95mm_HandSolder, F.Cu at (168.2, 67.8)
- added R13: 10k 1%, Resistor_SMD:R_0603_1608Metric_Pad0.98x0.95mm_HandSolder, F.Cu at (179.2, 68.0)
- added R14: 10k 1%, Resistor_SMD:R_0603_1608Metric_Pad0.98x0.95mm_HandSolder, F.Cu at (179.3, 73.7)
- added R15: 10k 1%, Resistor_SMD:R_0603_1608Metric_Pad0.98x0.95mm_HandSolder, F.Cu at (173.6, 62.8)
- added R16: 10k 1%, Resistor_SMD:R_0603_1608Metric_Pad0.98x0.95mm_HandSolder, F.Cu at (175.3, 68.8)
- added R17: 3.3k 1%, Resistor_SMD:R_0603_1608Metric_Pad0.98x0.95mm_HandSolder, F.Cu at (155.0, 87.2)
- added R18: 3.3k 1%, Resistor_SMD:R_0603_1608Metric_Pad0.98x0.95mm_HandSolder, F.Cu at (158.1, 91.4)
- added R19: 1.6k 1%, Resistor_SMD:R_0603_1608Metric_Pad0.98x0.95mm_HandSolder, F.Cu at (155.9, 81.3)
- added R2: 3.3k 1%, Resistor_SMD:R_0603_1608Metric_Pad0.98x0.95mm_HandSolder, F.Cu at (151.1, 65.9)
- added R20: 1.6k 1%, Resistor_SMD:R_0603_1608Metric_Pad0.98x0.95mm_HandSolder, F.Cu at (158.1, 86.2)
- added R21: 64.9k 1%, Resistor_SMD:R_0603_1608Metric_Pad0.98x0.95mm_HandSolder, F.Cu at (153.6, 75.3)
- added R22: 430 1%, Resistor_SMD:R_0603_1608Metric_Pad0.98x0.95mm_HandSolder, F.Cu at (155.2, 75.3)
- added R23: 64.9k 1%, Resistor_SMD:R_0603_1608Metric_Pad0.98x0.95mm_HandSolder, F.Cu at (153.7, 78.7)
- added R24: 430 1%, Resistor_SMD:R_0603_1608Metric_Pad0.98x0.95mm_HandSolder, F.Cu at (155.2, 78.7)
- added R25: 200k 1%, Resistor_SMD:R_0603_1608Metric_Pad0.98x0.95mm_HandSolder, F.Cu at (164.9, 79.5)
- added R26: 200k 1%, Resistor_SMD:R_0603_1608Metric_Pad0.98x0.95mm_HandSolder, F.Cu at (168.2, 75.9)
- added R27: 1k 1%, Resistor_SMD:R_0603_1608Metric_Pad0.98x0.95mm_HandSolder, F.Cu at (166.6, 79.5)
- added R28: 1k 1%, Resistor_SMD:R_0603_1608Metric_Pad0.98x0.95mm_HandSolder, F.Cu at (168.2, 79.5)
- added R29: 10k 1%, Resistor_SMD:R_0603_1608Metric_Pad0.98x0.95mm_HandSolder, F.Cu at (178.9, 79.4)
- added R3: 1.6k 1%, Resistor_SMD:R_0603_1608Metric_Pad0.98x0.95mm_HandSolder, F.Cu at (156.8, 61.4)
- added R30: 10k 1%, Resistor_SMD:R_0603_1608Metric_Pad0.98x0.95mm_HandSolder, F.Cu at (178.9, 85.3)
- added R31: 10k 1%, Resistor_SMD:R_0603_1608Metric_Pad0.98x0.95mm_HandSolder, F.Cu at (175.3, 74.6)
- added R32: 10k 1%, Resistor_SMD:R_0603_1608Metric_Pad0.98x0.95mm_HandSolder, F.Cu at (175.1, 80.9)
- added R33: 10k, Resistor_SMD:R_0603_1608Metric_Pad0.98x0.95mm_HandSolder, F.Cu at (167.7, 105.9)
- added R34: 20k, Resistor_SMD:R_0603_1608Metric_Pad0.98x0.95mm_HandSolder, F.Cu at (167.7, 107.6)
- added R35: 10k, Resistor_SMD:R_0603_1608Metric_Pad0.98x0.95mm_HandSolder, F.Cu at (167.7, 101.0)
- added R36: 20k, Resistor_SMD:R_0603_1608Metric_Pad0.98x0.95mm_HandSolder, F.Cu at (167.7, 102.7)
- added R37: 0R, Resistor_SMD:R_0603_1608Metric_Pad0.98x0.95mm_HandSolder, F.Cu at (182.5, 106.3)
- added R38: 0R, Resistor_SMD:R_0603_1608Metric_Pad0.98x0.95mm_HandSolder, F.Cu at (182.5, 108.0)
- added R39: 0R, Resistor_SMD:R_0603_1608Metric_Pad0.98x0.95mm_HandSolder, F.Cu at (182.5, 101.0)
- added R4: 1.6k 1%, Resistor_SMD:R_0603_1608Metric_Pad0.98x0.95mm_HandSolder, F.Cu at (156.8, 64.9)
- added R40: 0R, Resistor_SMD:R_0603_1608Metric_Pad0.98x0.95mm_HandSolder, F.Cu at (182.5, 102.5)
- added R41: 1k 1%, Resistor_SMD:R_0603_1608Metric_Pad0.98x0.95mm_HandSolder, F.Cu at (167.6, 109.3)
- added R42: 1k 1%, Resistor_SMD:R_0603_1608Metric_Pad0.98x0.95mm_HandSolder, F.Cu at (167.7, 99.2)
- added R43: 15 1%, Resistor_SMD:R_0603_1608Metric_Pad0.98x0.95mm_HandSolder, F.Cu at (170.2, 110.0)
- added R44: 15 1%, Resistor_SMD:R_0603_1608Metric_Pad0.98x0.95mm_HandSolder, F.Cu at (170.2, 98.7)
- added R45: 1.5M 1%, Resistor_SMD:R_0603_1608Metric_Pad0.98x0.95mm_HandSolder, F.Cu at (177.4, 110.8)
- added R46: 1.5M 1%, Resistor_SMD:R_0603_1608Metric_Pad0.98x0.95mm_HandSolder, F.Cu at (177.5, 98.0)
- added R47: 10k 1%, Resistor_SMD:R_0603_1608Metric_Pad0.98x0.95mm_HandSolder, F.Cu at (176.5, 113.6)
- added R48: 10k 1%, Resistor_SMD:R_0603_1608Metric_Pad0.98x0.95mm_HandSolder, F.Cu at (176.6, 95.3)
- added R49: 300k 1%, Resistor_SMD:R_0603_1608Metric_Pad0.98x0.95mm_HandSolder, F.Cu at (146.3, 87.2)
- added R5: 64.9k 1%, Resistor_SMD:R_0603_1608Metric_Pad0.98x0.95mm_HandSolder, F.Cu at (153.7, 71.9)
- added R50: 71.5k 1%, Resistor_SMD:R_0603_1608Metric_Pad0.98x0.95mm_HandSolder, F.Cu at (147.0, 84.7)
- added R51: 100k 1%, Resistor_SMD:R_0603_1608Metric_Pad0.98x0.95mm_HandSolder, F.Cu at (147.9, 82.2)
- added R6: 430 1%, Resistor_SMD:R_0603_1608Metric_Pad0.98x0.95mm_HandSolder, F.Cu at (155.2, 71.9)
- added R7: 64.9k 1%, Resistor_SMD:R_0603_1608Metric_Pad0.98x0.95mm_HandSolder, F.Cu at (153.7, 68.5)
- added R8: 430 1%, Resistor_SMD:R_0603_1608Metric_Pad0.98x0.95mm_HandSolder, F.Cu at (155.2, 68.5)
- added R9: 200k 1%, Resistor_SMD:R_0603_1608Metric_Pad0.98x0.95mm_HandSolder, F.Cu at (164.9, 67.7)
- added RS1: 10 0.5W 1%, Resistor_SMD:R_1210_3225Metric_Pad1.30x2.65mm_HandSolder, F.Cu at (174.4, 65.5)
- added RS2: 10 0.5W 1%, Resistor_SMD:R_1210_3225Metric_Pad1.30x2.65mm_HandSolder, F.Cu at (174.5, 71.2)
- added RS3: 10 0.5W 1%, Resistor_SMD:R_1210_3225Metric_Pad1.30x2.65mm_HandSolder, F.Cu at (174.5, 77.0)
- added RS4: 10 0.5W 1%, Resistor_SMD:R_1210_3225Metric_Pad1.30x2.65mm_HandSolder, F.Cu at (174.5, 83.9)
- added U2: MCP6242T-E/SN, Package_SO:SOIC-8_3.9x4.9mm_P1.27mm, F.Cu at (160.9, 65.6)
- added U3: LM339B, Package_SO:SOIC-14_3.9x8.7mm_P1.27mm, F.Cu at (162.8, 73.5)
- added U4: MCP6242T-E/SN, Package_SO:SOIC-8_3.9x4.9mm_P1.27mm, F.Cu at (160.9, 81.5)
- added U5: MCP6242T-E/SN, Package_SO:SOIC-8_3.9x4.9mm_P1.27mm, F.Cu at (172.1, 104.3)
- added U6: TLV9142, Package_SO:SOIC-8_3.9x4.9mm_P1.27mm, F.Cu at (177.9, 104.3)
- added U7: TPS7A4901DGNR, kml-custom:DGN8_1P89X1P57, F.Cu at (140.9, 85.2)
Connections:
- A1 pad 12: unconnected-(A1-D9-Pad12) -> /PWM2
- A1 pad 13: unconnected-(A1-D10-Pad13) -> /PWM3
- A1 pad 14: unconnected-(A1-D11-Pad14) -> /PWM4
- A1 pad 19: unconnected-(A1-A0-Pad19) -> /PD1
- A1 pad 20: unconnected-(A1-A1-Pad20) -> /PD2
- A1 pad 9: unconnected-(A1-D6-Pad9) -> /PWM1
Routing:
- net +5VA: track 0.00 -> 176.0 mm, vias 0 -> 9
- net GNDA: track 0.00 -> 82.0 mm, vias 0 -> 38
- net /PWM2: track 0.00 -> 63.0 mm, vias 0 -> 1
- net /PWM1: track 0.00 -> 59.7 mm, vias 0 -> 1
- net /PWM4: track 0.00 -> 46.8 mm, vias 0 -> 1
- net /PWM3: track 0.00 -> 45.1 mm, vias 0 -> 1
- net /PD2: track 0.00 -> 41.6 mm
- net /Linear Constant‐Current LED Driver x4/DAC_4: track 0.00 -> 26.0 mm, vias 0 -> 2
- net GND: track 16.8 -> 41.7 mm
- net /PD1: track 0.00 -> 24.9 mm
- net /Linear Constant‐Current LED Driver x4/FEEDBACK_2: track 0.00 -> 23.9 mm
- net /Linear Constant‐Current LED Driver x4/DAC_1: track 0.00 -> 22.6 mm, vias 0 -> 2
- net /Linear Constant‐Current LED Driver x4/DAC_2: track 0.00 -> 21.7 mm, vias 0 -> 2
- net /Linear Constant‐Current LED Driver x4/FEEDBACK_3: track 0.00 -> 20.8 mm
- net /Linear Constant‐Current LED Driver x4/DAC_3: track 0.00 -> 20.8 mm
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- added copper zone on B.Cu, net GNDA
Other:
- board text added: "BREAD Slice LED-PD Photometer SLC_LEPD R3 04-2025"
- board text added: "LED1"
- board text added: "LED2"
- board text added: "LED3"
- board text added: "LED4"
- board text added: "PD1"
- board text added: "PD2"
- board text removed: "BREAD Slice Template SLC_TEMP R3 04-2025"
