File: hardware/linear_cc_led_driver.kicad_sch (KiCad schematic)
At the start: 96 parts, among them Q1 BSS806NH6327XTSA1, Q2 BC858BWT1G, Q3 BC858BWT1G, Q4 BSS806NH6327XTSA1, Q5 BC858BWT1G, Q6 BSS806NH6327XTSA1, Q7 BC858BWT1G, Q8 BSS806NH6327XTSA1, U3 LM339B, U4 MCP6242T-E/SN, U5 MCP6242T-E/SN, U6 MCP6242T-E/SN

Commit message: finalized initial schematic and board
Parts:
- removed U6: MCP6242T-E/SN, Package_DFN_QFN:DFN-8-1EP_3x2mm_P0.5mm_EP1.75x1.45mm, symbol Amplifier_Operational:MCP6002-xMC
- C10, C11, C16, C7: footprint (none) -> Capacitor_SMD:C_0603_1608Metric_Pad1.08x0.95mm_HandSolder
- C12: renamed from C14; footprint (none) -> Capacitor_SMD:C_0603_1608Metric_Pad1.08x0.95mm_HandSolder
- C13: renamed from C12; footprint (none) -> Capacitor_SMD:C_0603_1608Metric_Pad1.08x0.95mm_HandSolder
- C14: renamed from C15; footprint (none) -> Capacitor_SMD:C_0603_1608Metric_Pad1.08x0.95mm_HandSolder
- C15: renamed from C13; footprint (none) -> Capacitor_SMD:C_0603_1608Metric_Pad1.08x0.95mm_HandSolder
- C5: renamed from C6; footprint (none) -> Capacitor_SMD:C_0603_1608Metric_Pad1.08x0.95mm_HandSolder
- C6: renamed from C8; footprint (none) -> Capacitor_SMD:C_0603_1608Metric_Pad1.08x0.95mm_HandSolder
- C8: renamed from C9; footprint (none) -> Capacitor_SMD:C_0603_1608Metric_Pad1.08x0.95mm_HandSolder
- C9: renamed from C5; footprint (none) -> Capacitor_SMD:C_0603_1608Metric_Pad1.08x0.95mm_HandSolder
- D10: renamed from D4; footprint SOD-923_TOS -> Diode_SMD:D_SOD-923
- D11: renamed from D5; footprint SOD-923_TOS -> Diode_SMD:D_SOD-923
- D8: renamed from D2; footprint SOD-923_TOS -> Diode_SMD:D_SOD-923
- D9: renamed from D3; footprint SOD-923_TOS -> Diode_SMD:D_SOD-923
- R1: renamed from R8; footprint (none) -> Resistor_SMD:R_0603_1608Metric_Pad0.98x0.95mm_HandSolder
- R10: renamed from R13; footprint (none) -> Resistor_SMD:R_0603_1608Metric_Pad0.98x0.95mm_HandSolder
- R11: renamed from R4; footprint (none) -> Resistor_SMD:R_0603_1608Metric_Pad0.98x0.95mm_HandSolder
- R12: renamed from R14; footprint (none) -> Resistor_SMD:R_0603_1608Metric_Pad0.98x0.95mm_HandSolder
- R13: renamed from R6; footprint (none) -> Resistor_SMD:R_0603_1608Metric_Pad0.98x0.95mm_HandSolder
- R14: renamed from R15; footprint (none) -> Resistor_SMD:R_0603_1608Metric_Pad0.98x0.95mm_HandSolder
- R15: renamed from R5; footprint (none) -> Resistor_SMD:R_0603_1608Metric_Pad0.98x0.95mm_HandSolder
- R16, R17, R32: footprint (none) -> Resistor_SMD:R_0603_1608Metric_Pad0.98x0.95mm_HandSolder
- R18: renamed from R25; footprint (none) -> Resistor_SMD:R_0603_1608Metric_Pad0.98x0.95mm_HandSolder
- R19: renamed from R18; footprint (none) -> Resistor_SMD:R_0603_1608Metric_Pad0.98x0.95mm_HandSolder
- R2: renamed from R9; footprint (none) -> Resistor_SMD:R_0603_1608Metric_Pad0.98x0.95mm_HandSolder
- R20: renamed from R26; footprint (none) -> Resistor_SMD:R_0603_1608Metric_Pad0.98x0.95mm_HandSolder
- R21: renamed from R19; footprint (none) -> Resistor_SMD:R_0603_1608Metric_Pad0.98x0.95mm_HandSolder
- R22: renamed from R20; footprint (none) -> Resistor_SMD:R_0603_1608Metric_Pad0.98x0.95mm_HandSolder
- R23: renamed from R27; footprint (none) -> Resistor_SMD:R_0603_1608Metric_Pad0.98x0.95mm_HandSolder
- R24: renamed from R28; footprint (none) -> Resistor_SMD:R_0603_1608Metric_Pad0.98x0.95mm_HandSolder
- R25: renamed from R21; footprint (none) -> Resistor_SMD:R_0603_1608Metric_Pad0.98x0.95mm_HandSolder
- R26: renamed from R29; footprint (none) -> Resistor_SMD:R_0603_1608Metric_Pad0.98x0.95mm_HandSolder
- R27: renamed from R22; footprint (none) -> Resistor_SMD:R_0603_1608Metric_Pad0.98x0.95mm_HandSolder
- R28: renamed from R30; footprint (none) -> Resistor_SMD:R_0603_1608Metric_Pad0.98x0.95mm_HandSolder
- R29: renamed from R23; footprint (none) -> Resistor_SMD:R_0603_1608Metric_Pad0.98x0.95mm_HandSolder
- R3: renamed from R7; footprint (none) -> Resistor_SMD:R_0603_1608Metric_Pad0.98x0.95mm_HandSolder
- R30: renamed from R31; footprint (none) -> Resistor_SMD:R_0603_1608Metric_Pad0.98x0.95mm_HandSolder
- R31: renamed from R24; footprint (none) -> Resistor_SMD:R_0603_1608Metric_Pad0.98x0.95mm_HandSolder
- R4: renamed from R10; footprint (none) -> Resistor_SMD:R_0603_1608Metric_Pad0.98x0.95mm_HandSolder
- R5: renamed from R1; footprint (none) -> Resistor_SMD:R_0603_1608Metric_Pad0.98x0.95mm_HandSolder
- R6: renamed from R2; footprint (none) -> Resistor_SMD:R_0603_1608Metric_Pad0.98x0.95mm_HandSolder
- R7: renamed from R11; footprint (none) -> Resistor_SMD:R_0603_1608Metric_Pad0.98x0.95mm_HandSolder
- R8: renamed from R12; footprint (none) -> Resistor_SMD:R_0603_1608Metric_Pad0.98x0.95mm_HandSolder
- R9: renamed from R3; footprint (none) -> Resistor_SMD:R_0603_1608Metric_Pad0.98x0.95mm_HandSolder
- RS1, RS2, RS3, RS4: footprint (none) -> Resistor_SMD:R_1210_3225Metric_Pad1.30x2.65mm_HandSolder
- TP1, TP15, TP16, TP17, TP31, TP32: footprint (none) -> TestPoint:TestPoint_Keystone_5000-5004_Miniature
- TP10: renamed from TP4; footprint (none) -> TestPoint:TestPoint_Keystone_5000-5004_Miniature
- TP11: renamed from TP13; footprint (none) -> TestPoint:TestPoint_Keystone_5000-5004_Miniature
- TP12: renamed from TP14; footprint (none) -> TestPoint:TestPoint_Keystone_5000-5004_Miniature
- TP13: renamed from TP5; footprint (none) -> TestPoint:TestPoint_Keystone_5000-5004_Miniature
- TP14: renamed from TP6; footprint (none) -> TestPoint:TestPoint_Keystone_5000-5004_Miniature
- TP18: renamed from TP25; footprint (none) -> TestPoint:TestPoint_Keystone_5000-5004_Miniature
- TP19: renamed from TP18; footprint (none) -> TestPoint:TestPoint_Keystone_5000-5004_Miniature
- TP2: renamed from TP9; footprint (none) -> TestPoint:TestPoint_Keystone_5000-5004_Miniature
- TP20: renamed from TP19; footprint (none) -> TestPoint:TestPoint_Keystone_5000-5004_Miniature
- TP21: renamed from TP20; footprint (none) -> TestPoint:TestPoint_Keystone_5000-5004_Miniature
- TP22: renamed from TP26; footprint (none) -> TestPoint:TestPoint_Keystone_5000-5004_Miniature
- TP23: renamed from TP27; footprint (none) -> TestPoint:TestPoint_Keystone_5000-5004_Miniature
- TP24: renamed from TP28; footprint (none) -> TestPoint:TestPoint_Keystone_5000-5004_Miniature
- TP25: renamed from TP21; footprint (none) -> TestPoint:TestPoint_Keystone_5000-5004_Miniature
- TP26: renamed from TP22; footprint (none) -> TestPoint:TestPoint_Keystone_5000-5004_Miniature
- TP27: renamed from TP29; footprint (none) -> TestPoint:TestPoint_Keystone_5000-5004_Miniature
- TP28: renamed from TP30; footprint (none) -> TestPoint:TestPoint_Keystone_5000-5004_Miniature
- TP29: renamed from TP23; footprint (none) -> TestPoint:TestPoint_Keystone_5000-5004_Miniature
- TP3: renamed from TP8; footprint (none) -> TestPoint:TestPoint_Keystone_5000-5004_Miniature
- TP30: renamed from TP24; footprint (none) -> TestPoint:TestPoint_Keystone_5000-5004_Miniature
- TP4: renamed from TP2; footprint (none) -> TestPoint:TestPoint_Keystone_5000-5004_Miniature
- TP5: renamed from TP3; footprint (none) -> TestPoint:TestPoint_Keystone_5000-5004_Miniature
- TP6: renamed from TP10; footprint (none) -> TestPoint:TestPoint_Keystone_5000-5004_Miniature
- TP7: renamed from TP11; footprint (none) -> TestPoint:TestPoint_Keystone_5000-5004_Miniature
- TP8: renamed from TP12; footprint (none) -> TestPoint:TestPoint_Keystone_5000-5004_Miniature
- TP9: renamed from TP7; footprint (none) -> TestPoint:TestPoint_Keystone_5000-5004_Miniature
- U2: renamed from U4; footprint Package_DFN_QFN:DFN-8-1EP_3x2mm_P0.5mm_EP1.75x1.45mm -> Package_SO:SOIC-8_3.9x4.9mm_P1.27mm
- U3: footprint (none) -> Package_SO:SOIC-14_3.9x8.7mm_P1.27mm
- U4: renamed from U5; footprint Package_DFN_QFN:DFN-8-1EP_3x2mm_P0.5mm_EP1.75x1.45mm -> Package_SO:SOIC-8_3.9x4.9mm_P1.27mm
- renumbered Q2 to Q1, Q1 to Q2
Connections:
- net COMP_REF_2: now also U3.6 (-); no longer U3.7 (+)
- net COMP_REF_3: now also U3.10 (-); no longer U3.11 (+)
- net COMP_REF_4: now also U3.8 (-); no longer U3.9 (+)
- net DAC_1: no longer C11.1, C12.1, C13.1, C14.1, R17.2, R18.2, R19.1, R20.1, R25.1, R26.1, U3.10 (-), U3.8 (-), U4.3 (+), U4.5 (+)
- net DAC_2: now also U3.7 (+); no longer U3.6 (-)
- net +5VA renamed +5V
- net GNDA renamed GND
- new net DAC_3: C11.1, C13.1, R17.2, R19.1, R25.1, U3.11 (+), U4.3 (+)
- new net DAC_4: C12.1, C14.1, R18.2, R20.1, R26.1, U3.9 (+), U4.5 (+)
